Commit message: update urdf and ros2 visualization pkg

File: src/ros2_ws/src/rover_description/urdf/pragyaan_rover.urdf (robot description, URDF)
Before this commit: robot pragyaan_rover, 14 links, 13 joints
Links:
- link Wheel_back_left: geometry collision mesh filename=package://rover_description/meshes/Wheel_back_left_Circle_0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 scale=2 1 1; visual mesh filename=package://rover_description/meshes/Wheel_back_left_Circle_0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 scale=2 1 1
- link Wheel_back_right: geometry collision mesh filename=package://rover_description/meshes/Wheel_back_right_Circle_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 scale=2 1 1; visual mesh filename=package://rover_description/meshes/Wheel_back_right_Circle_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 scale=2 1 1
- link Wheel_front_left: geometry collision mesh filename=package://rover_description/meshes/Wheel_front_left_Circle_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 scale=2 1 1; visual mesh filename=package://rover_description/meshes/Wheel_front_left_Circle_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 scale=2 1 1
- link Wheel_front_right: geometry collision mesh filename=package://rover_description/meshes/Wheel_front_right_Circle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 scale=2 1 1; visual mesh filename=package://rover_description/meshes/Wheel_front_right_Circle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 scale=2 1 1
- link Wheel_middle_left: geometry collision mesh filename=package://rover_description/meshes/Wheel_middle_left_Circle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 scale=2 1 1; visual mesh filename=package://rover_description/meshes/Wheel_middle_left_Circle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 scale=2 1 1
- link Wheel_middle_right: geometry collision mesh filename=package://rover_description/meshes/Wheel_middle_right_Circl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 scale=2 1 1; visual mesh filename=package://rover_description/meshes/Wheel_middle_right_Circl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 scale=2 1 1

Commit message: adding dummy of pragyaan to isaacsim

File: src/ros2_ws/src/rover_description/urdf/pragyaan_rover.urdf (robot description, URDF)
Before this commit: robot pragyaan_rover, 14 links, 13 joints
Links:
- added link base_link
Joints:
- added joint base_body_joint: type fixed, parent base_link, child Pragyaan, origin xyz=0 0 0 rpy=1.571 0 0
